File: retro-game-console.kicad_sch (KiCad schematic)
At the start: 3 parts, among them U1 ESP32-DevKitC, U2 LCD_ILI9341, U3 Catalex_Micro_SD

Commit message: Progress
Parts:
- removed U2: LCD_ILI9341, JS_Displays:LCD_ILI9341, symbol JS_Displays:LCD_ILI9341
- removed U3: Catalex_Micro_SD, TZXDuino:Catalex_Micro_SD, symbol TZXDuino:Catalex_Micro_SD
- added C1: C104, Capacitor_THT:C_Rect_L7.0mm_W3.5mm_P5.00mm, symbol Device:C
- added D1: LED, symbol Device:LED
- added LS1: Speaker, RGC_Components:Speaker, symbol Device:Speaker
- added R1: R220, LED_THT:LED_D5.0mm, symbol Device:R
- added R2, R4, R5: R10K, LED_THT:LED_D5.0mm, symbol Device:R
- added R3: R1K, symbol Device:R
- added SW1, SW2: SW_Push, Button_Switch_THT:SW_PUSH_6mm_H5mm, symbol Switch:SW_Push
- added U2: Battery_shield_v3, RGC_Components:Battery_shield_v3, symbol RGC_Components:Battery_shield_v3
- added U3: Micro_SD_card_adapter, RGC_Components:Micro_SD_card_adapter, symbol RGC_Components:Micro_SD_card_adapter
- added U4: MAX98357A_Breakout, RGC_Components:MAX98357A_Breakout, symbol RGC_Components:MAX98357A_Breakout
- added U5: LCD_ILI9341, RGC_Components:LCD_2.4in, symbol JS_Displays:LCD_ILI9341
- added U6: 74HC165, symbol 74xx:74HC165
Connections:
- net +3.3V: now reaches U1.1 (3V3)
- net +3.3V: now also C1.2, R2.1, R4.2, R5.2, U2.1 (+3V), U3.2 (VCC), U4.1 (VCC), U5.14 (VCC), U6.16 (VCC)
- net AUD_BCLK: now reaches U1.10 (DAC_2/ADC2_CH9/GPIO26)
- net AUD_BCLK: now also U4.4 (BCLK)
- net AUD_LRC: now reaches U1.11 (ADC2_CH7/GPIO27)
- net AUD_LRC: now also U4.3 (LRC)
- net LCD_SCK: now reaches U1.12 (MTMS/GPIO14/ADC2_CH6)
- net LCD_SCK: now also U5.8 (SCK)
- net LCD_BCKL: now reaches U1.13 (*MTDI/GPIO12/ADC2_CH5)
- net LCD_BCKL: now also R3.1
- net LCD_MOSI: now reaches U1.15 (MTCK/GPIO13/ADC2_CH4)
- net LCD_MOSI: now also U5.9 (MOSI)
- net LCD_CS: now reaches U1.23 (*MTDO/GPIO15/ADC2_CH3)
- net LCD_CS: now also U5.12 (CS)
- net LCD_DC: now reaches U1.24 (ADC2_CH2/*GPIO2)
- net LCD_DC: now also U5.10 (D/C)
- net BTN_MENU: now reaches U1.26 (ADC2_CH0/GPIO4)
- net BTN_MENU: now also R4.1, SW1.1
- net BTN_OPTION: now reaches U1.29 (*GPIO5)
- net BTN_OPTION: now also R5.1, SW2.1
- net BAT_LEVEL: now reaches U1.3 (SENSOR_VP/GPIO36/ADC1_CH0)
- net SD_SCK: now reaches U1.30 (GPIO18)
- net SD_SCK: now also U3.5 (SCK)
- net SD_MISO: now reaches U1.31 (GPIO19)
- net SD_MISO: now also U3.3 (MISO)
- net LED_PIN: now reaches U1.33 (GPIO21)
- net LED_PIN: now also D1.2 (A)
- net SD_CS: now reaches U1.36 (GPIO22)
- net SD_CS: now also U3.6 (CS)
- net SD_MOSI: now reaches U1.37 (GPIO23)
- net SD_MOSI: now also U3.4 (MOSI)
- net GND: now reaches U1.38 (GND)
- net GND: now also C1.1, R1.2, SW1.2, SW2.2, U2.2 (GND), U3.1 (GND), U4.2 (GND), U4.6 (GAIN), U5.13 (GND), U6.8 (GND)
- net GAMEPAD_DATA: now reaches U1.6 (VDET_2/GPIO35/ADC1_CH7)
- net GAMEPAD_LATCH: now reaches U1.7 (32K_XP/GPIO32/ADC1_CH4)
- net GAMEPAD_CLOCK: now reaches U1.8 (32K_XN/GPIO33/ADC1_CH5)
- net AUD_DIN: now reaches U1.9 (DAC_1/ADC2_CH8/GPIO25)
- net AUD_DIN: now also U4.5 (DIN)
- new net: D1.1 (K), R1.1
- new net: LS1.1, U4.8 (AUDIO_POS)
- new net: LS1.2, U4.9 (AUDIO_NEG)
- new net LCD_BCKL_OUT: R3.2, U5.7 (LED)
- new net LCD_RESET: R2.2, U5.11 (RESET)
- no-connect marks 0 -> 28
Other:
- moved on the sheet: U1

Commit message: Schema done
Parts:
- added C2, C3: C104, Capacitor_THT:C_Rect_L7.0mm_W3.5mm_P5.00mm, symbol Device:C
- added J1: Battery_Clip, Connector_PinSocket_2.54mm:PinSocket_1x01_P2.54mm_Vertical, symbol Connector:Conn_01x01_Female
- added R10, R11, R12, R9: R1K, Resistor_THT:R_Axial_DIN0309_L9.0mm_D3.2mm_P12.70mm_Horizontal, symbol Device:R
- added R13, R14, R15, R16, R17, R18, R19, R20, R6, R7, R8: R10K, Resistor_THT:R_Axial_DIN0309_L9.0mm_D3.2mm_P12.70mm_Horizontal, symbol Device:R
- added SW_A1, SW_SELECT1, SW_START1: SW_Push, Button_Switch_SMD:SW_Push_1P1T_NO_6x6mm_H9.5mm, symbol Switch:SW_Push
- added SW_B1, SW_DOWN1, SW_LEFT1, SW_RIGHT1, SW_UP1: SW_Push, Button_Switch_THT:SW_PUSH-12mm, symbol Switch:SW_Push
- D1: footprint (none) -> LED_THT:LED_D5.0mm
- R1: value R220 -> R1K; footprint LED_THT:LED_D5.0mm -> Resistor_THT:R_Axial_DIN0309_L9.0mm_D3.2mm_P12.70mm_Horizontal
- R2, R4, R5: footprint LED_THT:LED_D5.0mm -> Resistor_THT:R_Axial_DIN0309_L9.0mm_D3.2mm_P12.70mm_Horizontal
- R3: footprint (none) -> Resistor_THT:R_Axial_DIN0309_L9.0mm_D3.2mm_P12.70mm_Horizontal
- SW_MENU1: renamed from SW1; footprint Button_Switch_THT:SW_PUSH_6mm_H5mm -> Button_Switch_SMD:SW_Push_1P1T_NO_6x6mm_H9.5mm
- SW_OPTION1: renamed from SW2; footprint Button_Switch_THT:SW_PUSH_6mm_H5mm -> Button_Switch_SMD:SW_Push_1P1T_NO_6x6mm_H9.5mm
Connections:
- net +3.3V: now also C3.2, R13.2, R14.2, R15.2, R16.2, R17.2, R18.2, R19.2, R20.2; no longer U2.1 (+3V)
- net BAT_LEVEL: now also C2.2, R7.1, R8.2
- net GAMEPAD_CLOCK: now also R11.1
- net GAMEPAD_DATA: now also R12.2
- net GAMEPAD_LATCH: now also R10.1
- net GND: now also U6.10 (DS), U6.15 (~{CE}), C2.1, C3.1, R8.1, SW_A1.2, SW_B1.2, SW_DOWN1.2, SW_LEFT1.2, SW_RIGHT1.2, SW_SELECT1.2, SW_START1.2, SW_UP1.2; no longer U2.2 (GND)
- net LCD_DC: now also R9.1; no longer U5.10 (D/C)
- net at U6.1 (~{PL}): now also R10.2
- net BTN_UP: now reaches U6.11 (D0)
- net BTN_UP: now also R13.1, SW_UP1.1
- net BTN_RIGHT: now reaches U6.12 (D1)
- net BTN_RIGHT: now also R16.1, SW_RIGHT1.1
- net BTN_DOWN: now reaches U6.13 (D2)
- net BTN_DOWN: now also R14.1, SW_DOWN1.1
- net BTN_LEFT: now reaches U6.14 (D3)
- net BTN_LEFT: now also R15.1, SW_LEFT1.1
- net at U6.2 (CP): now also R11.2
- net BTN_SELECT: now reaches U6.3 (D4)
- net BTN_SELECT: now also R17.1, SW_SELECT1.1
- net BTN_START: now reaches U6.4 (D5)
- net BTN_START: now also R19.1, SW_START1.1
- net BTN_A: now reaches U6.5 (D6)
- net BTN_A: now also R18.1, SW_A1.1
- net BTN_B: now reaches U6.6 (D7)
- net BTN_B: now also R20.1, SW_B1.1
- net at U6.7 (~{Q7}): now also R12.1
- new net: R6.1, R7.2
- new net: J1.1 (Pin_1), R6.2
- new net LCD_DC_OUT: R9.2, U5.10 (D/C)
- no-connect marks 28 -> 31
Other:
- moved on the sheet: C1, D1, LS1, R1, R2, R3, R4, R5, SW_MENU1, SW_OPTION1, U1, U3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
