File: retro-game-console.kicad_sch (KiCad schematic)
At the start: 42 parts, among them J1 Battery_Clip, U1 ESP32-DevKitC, U2 Battery_shield_v3, U3 Micro_SD_card_adapter, U4 MAX98357A_Breakout, U5 LCD_ILI9341, U6 74HC165

Commit message: Network in progress
Parts:
- removed U2: Battery_shield_v3, RGC_Components:Battery_shield_v3, symbol RGC_Components:Battery_shield_v3
- added U1: Battery_shield_v3, RGC_Components:Battery_shield_v3, symbol RGC_Components:Battery_shield_v3
- R13, R14, R15: footprint Resistor_THT:R_Axial_DIN0309_L9.0mm_D3.2mm_P12.70mm_Horizontal -> Resistor_THT:R_Axial_DIN0309_L9.0mm_D3.2mm_P15.24mm_Horizontal
- SW_A1: footprint Button_Switch_SMD:SW_Push_1P1T_NO_6x6mm_H9.5mm -> Button_Switch_THT:SW_PUSH-12mm
- U6: footprint (none) -> Package_DIP:DIP-16_W7.62mm_LongPads
Connections:
- no-connect marks 31 -> 29
Changed lines of the file:
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@@
   (no_connect (at 165.1 74.93))
   (no_connect (at 165.1 72.39))
-  (no_connect (at 31.75 26.67))
-  (no_connect (at 48.26 26.67))
   (no_connect (at 96.52 67.31))
   (no_connect (at 96.52 72.39))
@@
       (effects (font (size 1.27 1.27)) (justify right))
     )
-    (property "Footprint" "Resistor_THT:R_Axial_DIN0309_L9.0mm_D3.2mm_P12.70mm_Horizontal" (id 2) (at 260.858 43.18 90)
+    (property "Footprint" "Resistor_THT:R_Axial_DIN0309_L9.0mm_D3.2mm_P15.24mm_Horizontal" (id 2) (at 260.858 43.18 90)
       (effects (font (size 1.27 1.27)) hide)
     )
@@
     (property "Reference" "SW_A1" (id 0) (at 267.97 82.55 0))
     (property "Value" "SW_Push" (id 1) (at 267.97 85.09 0))
-    (property "Footprint" "Button_Switch_SMD:SW_Push_1P1T_NO_6x6mm_H9.5mm" (id 2) (at 267.97 85.09 0)
+    (property "Footprint" "Button_Switch_THT:SW_PUSH-12mm" (id 2) (at 267.97 85.09 0)
       (effects (font (size 1.27 1.27)) hide)
     )
@@
       (effects (font (size 1.27 1.27)) (justify right))
     )
-    (property "Footprint" "Resistor_THT:R_Axial_DIN0309_L9.0mm_D3.2mm_P12.70mm_Horizontal" (id 2) (at 215.138 62.23 90)
+    (property "Footprint" "Resistor_THT:R_Axial_DIN0309_L9.0mm_D3.2mm_P15.24mm_Horizontal" (id 2) (at 215.138 62.23 90)
       (effects (font (size 1.27 1.27)) hide)
     )
@@
     (pin "2")
   )
-  (symbol (lib_id "RGC_Components:Battery_shield_v3") (at 39.37 22.86 0) (unit 1)
-    (in_bom yes) (on_board yes) (fields_autoplaced)
-    (property "Reference" "U2" (id 0) (at 40.005 19.05 0))
-    (property "Value" "Battery_shield_v3" (id 1) (at 40.005 21.59 0))
-    (property "Footprint" "RGC_Components:Battery_shield_v3" (id 2) (at 36.83 22.86 0)
-      (effects (font (size 1.27 1.27)) hide)
-    )
-    (property "Datasheet" "" (id 3) (at 36.83 22.86 0)
-      (effects (font (size 1.27 1.27)) hide)
-    )
-    (pin "1")
-    (pin "2")
-  )
   (symbol (lib_id "power:GND") (at 233.68 90.17 0) (unit 1)
     (in_bom yes) (on_board yes) (fields_autoplaced)
@@
     (pin "1")
     (pin "2")
+  )
+  (symbol (lib_id "RGC_Components:Battery_shield_v3") (at 33.02 22.86 0) (unit 1)
+    (in_bom yes) (on_board yes) (fields_autoplaced)
+    (property "Reference" "U1" (id 0) (at 40.64 25.3999 0)
+      (effects (font (size 1.27 1.27)) (justify left))
+    )
+    (property "Value" "Battery_shield_v3" (id 1) (at 40.64 27.9399 0)
+      (effects (font (size 1.27 1.27)) (justify left))
+    )
+    (property "Footprint" "RGC_Components:Battery_shield_v3" (id 2) (at 30.48 22.86 0)
+      (effects (font (size 1.27 1.27)) hide)
+    )
+    (property "Datasheet" "" (id 3) (at 30.48 22.86 0)
+      (effects (font (size 1.27 1.27)) hide)
+    )
   )
   (symbol (lib_id "power:GND") (at 233.68 68.58 0) (unit 1)
@@
       (effects (font (size 1.27 1.27)) (justify left))
     )
-    (property "Footprint" "" (id 2) (at 140.97 152.4 0)
+    (property "Footprint" "Package_DIP:DIP-16_W7.62mm_LongPads" (id 2) (at 140.97 152.4 0)
       (effects (font (size 1.27 1.27)) hide)
     )
@@
       (effects (font (size 1.27 1.27)) (justify right))
     )
-    (property "Footprint" "Resistor_THT:R_Axial_DIN0309_L9.0mm_D3.2mm_P12.70mm_Horizontal" (id 2) (at 215.138 43.18 90)
+    (property "Footprint" "Resistor_THT:R_Axial_DIN0309_L9.0mm_D3.2mm_P15.24mm_Horizontal" (id 2) (at 215.138 43.18 90)
       (effects (font (size 1.27 1.27)) hide)
     )
@@
     )
     (path "/c3eb8f54-8621-41d8-bf4e-e4179e2e9d95"
-      (reference "R13") (unit 1) (value "R10K") (footprint "Resistor_THT:R_Axial_DIN0309_L9.0mm_D3.2mm_P12.70mm_Horizontal")
+      (reference "R13") (unit 1) (value "R10K") (footprint "Resistor_THT:R_Axial_DIN0309_L9.0mm_D3.2mm_P15.24mm_Horizontal")
     )
     (path "/073e876d-81ad-4fbd-875c-89e0d7a85c73"
-      (reference "R14") (unit 1) (value "R10K") (footprint "Resistor_THT:R_Axial_DIN0309_L9.0mm_D3.2mm_P12.70mm_Horizontal")
+      (reference "R14") (unit 1) (value "R10K") (footprint "Resistor_THT:R_Axial_DIN0309_L9.0mm_D3.2mm_P15.24mm_Horizontal")
     )
     (path "/327681b8-d06a-49ab-ade4-f813aa2a40b0"
-      (reference "R15") (unit 1) (value "R10K") (footprint "Resistor_THT:R_Axial_DIN0309_L9.0mm_D3.2mm_P12.70mm_Horizontal")
+      (reference "R15") (unit 1) (value "R10K") (footprint "Resistor_THT:R_Axial_DIN0309_L9.0mm_D3.2mm_P15.24mm_Horizontal")
     )
     (path "/7896e020-a247-4952-982c-204414362fdb"
@@
     )
     (path "/14ec2fba-b378-4d0b-b95a-ec2ddf937961"
-      (reference "SW_A1") (unit 1) (value "SW_Push") (footprint "Button_Switch_SMD:SW_Push_1P1T_NO_6x6mm_H9.5mm")
+      (reference "SW_A1") (unit 1) (value "SW_Push") (footprint "Button_Switch_THT:SW_PUSH-12mm")
     )
     (path "/1c19d6b4-e936-4dd5-a2af-785430f46541"
@@
       (reference "SW_UP1") (unit 1) (value "SW_Push") (footprint "Button_Switch_THT:SW_PUSH-12mm")
     )
+    (path "/98b5e36f-415d-4e64-b0c6-5f6e6d1487c3"
+      (reference "U1") (unit 1) (value "Battery_shield_v3") (footprint "RGC_Components:Battery_shield_v3")
+    )
     (path "/c44f4c1a-13b1-42c9-bf1b-c4ea764d2acb"
       (reference "U1") (unit 1) (value "ESP32-DevKitC") (footprint "Espressif:ESP32-DevKitC")
     )
-    (path "/43bede56-d715-420f-b3ee-fa8673af956b"
-      (reference "U2") (unit 1) (value "Battery_shield_v3") (footprint "RGC_Components:Battery_shield_v3")
-    )
     (path "/b2baff32-25b8-4dd9-b059-e0a76aa729b9"

Commit message: Before net
Parts:
- renumbered U1 to U2
Connections:
- net GND: now also D1.1 (K); no longer R1.2
- net LED_PIN: now also R1.1; no longer D1.2 (A)
- new net: D1.2 (A), R1.2
Other:
- moved on the sheet: D1, R1
Changed lines of the file:
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@@
-    (stroke (width 0) (type default) (color 0 0 0 0))
-  )
-  (wire (pts (xy 41.91 97.79) (xy 45.72 97.79))
     (stroke (width 0) (type default) (color 0 0 0 0))
   )
@@
     (stroke (width 0) (type default) (color 0 0 0 0))
   )
+  (wire (pts (xy 31.75 97.79) (xy 34.29 97.79))
+    (stroke (width 0) (type default) (color 0 0 0 0))
+  )
   (wire (pts (xy 213.36 30.48) (xy 217.17 30.48))
     (stroke (width 0) (type default) (color 0 0 0 0))
@@
     (stroke (width 0) (type default) (color 0 0 0 0))
   )
+  (wire (pts (xy 52.07 97.79) (xy 55.88 97.79))
+    (stroke (width 0) (type default) (color 0 0 0 0))
+  )
   (wire (pts (xy 227.33 109.22) (xy 233.68 109.22))
     (stroke (width 0) (type default) (color 0 0 0 0))
@@
     (stroke (width 0) (type default) (color 0 0 0 0))
   )
-  (wire (pts (xy 53.34 97.79) (xy 55.88 97.79))
-    (stroke (width 0) (type default) (color 0 0 0 0))
-  )
   (wire (pts (xy 165.1 95.25) (xy 168.91 95.25))
     (stroke (width 0) (type default) (color 0 0 0 0))
@@
     (stroke (width 0) (type default) (color 0 0 0 0))
   )
+  (wire (pts (xy 41.91 97.79) (xy 44.45 97.79))
+    (stroke (width 0) (type default) (color 0 0 0 0))
+  )
   (wire (pts (xy 140.97 177.8) (xy 140.97 179.07))
     (stroke (width 0) (type default) (color 0 0 0 0))
@@
   )
   (wire (pts (xy 259.08 46.99) (xy 259.08 49.53))
-    (stroke (width 0) (type default) (color 0 0 0 0))
-  )
-  (wire (pts (xy 31.75 97.79) (xy 34.29 97.79))
     (stroke (width 0) (type default) (color 0 0 0 0))
   )
@@
     (pin "1")
   )
-  (symbol (lib_id "Device:R") (at 49.53 97.79 90) (unit 1)
-    (in_bom yes) (on_board yes) (fields_autoplaced)
-    (property "Reference" "R1" (id 0) (at 49.53 91.44 90))
-    (property "Value" "R1K" (id 1) (at 49.53 93.98 90))
-    (property "Footprint" "Resistor_THT:R_Axial_DIN0309_L9.0mm_D3.2mm_P12.70mm_Horizontal" (id 2) (at 49.53 99.568 90)
-      (effects (font (size 1.27 1.27)) hide)
-    )
-    (property "Datasheet" "~" (id 3) (at 49.53 97.79 0)
-      (effects (font (size 1.27 1.27)) hide)
-    )
-    (pin "1")
-    (pin "2")
-  )
-  (symbol (lib_id "Device:LED") (at 38.1 97.79 180) (unit 1)
-    (in_bom yes) (on_board yes) (fields_autoplaced)
-    (property "Reference" "D1" (id 0) (at 39.6875 90.17 0))
-    (property "Value" "LED" (id 1) (at 39.6875 92.71 0))
-    (property "Footprint" "LED_THT:LED_D5.0mm" (id 2) (at 38.1 97.79 0)
+  (symbol (lib_id "Device:R") (at 38.1 97.79 90) (unit 1)
+    (in_bom yes) (on_board yes) (fields_autoplaced)
+    (property "Reference" "R1" (id 0) (at 38.1 91.44 90))
+    (property "Value" "R1K" (id 1) (at 38.1 93.98 90))
+    (property "Footprint" "Resistor_THT:R_Axial_DIN0309_L9.0mm_D3.2mm_P12.70mm_Horizontal" (id 2) (at 38.1 99.568 90)
       (effects (font (size 1.27 1.27)) hide)
     )
     (property "Datasheet" "~" (id 3) (at 38.1 97.79 0)
+      (effects (font (size 1.27 1.27)) hide)
+    )
+    (pin "1")
+    (pin "2")
+  )
+  (symbol (lib_id "Device:LED") (at 48.26 97.79 180) (unit 1)
+    (in_bom yes) (on_board yes) (fields_autoplaced)
+    (property "Reference" "D1" (id 0) (at 49.8475 90.17 0))
+    (property "Value" "LED" (id 1) (at 49.8475 92.71 0))
+    (property "Footprint" "LED_THT:LED_D5.0mm" (id 2) (at 48.26 97.79 0)
+      (effects (font (size 1.27 1.27)) hide)
+    )
+    (property "Datasheet" "~" (id 3) (at 48.26 97.79 0)
       (effects (font (size 1.27 1.27)) hide)
     )
@@
   (symbol (lib_id "RGC_Components:Battery_shield_v3") (at 33.02 22.86 0) (unit 1)
     (in_bom yes) (on_board yes) (fields_autoplaced)
-    (property "Reference" "U1" (id 0) (at 40.64 25.3999 0)
+    (property "Reference" "U2" (id 0) (at 40.64 25.3999 0)
       (effects (font (size 1.27 1.27)) (justify left))
     )
@@
       (reference "SW_UP1") (unit 1) (value "SW_Push") (footprint "Button_Switch_THT:SW_PUSH-12mm")
     )
-    (path "/98b5e36f-415d-4e64-b0c6-5f6e6d1487c3"
-      (reference "U1") (unit 1) (value "Battery_shield_v3") (footprint "RGC_Components:Battery_shield_v3")
-    )
     (path "/c44f4c1a-13b1-42c9-bf1b-c4ea764d2acb"
       (reference "U1") (unit 1) (value "ESP32-DevKitC") (footprint "Espressif:ESP32-DevKitC")
     )
+    (path "/98b5e36f-415d-4e64-b0c6-5f6e6d1487c3"
+      (reference "U2") (unit 1) (value "Battery_shield_v3") (footprint "RGC_Components:Battery_shield_v3")
+    )
     (path "/b2baff32-25b8-4dd9-b059-e0a76aa729b9"

Commit message: WIP
Parts:
- R18, R20: footprint Resistor_THT:R_Axial_DIN0309_L9.0mm_D3.2mm_P12.70mm_Horizontal -> Resistor_THT:R_Axial_DIN0309_L9.0mm_D3.2mm_P15.24mm_Horizontal
Changed lines of the file:
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@@
       (effects (font (size 1.27 1.27)) (justify right))
     )
-    (property "Footprint" "Resistor_THT:R_Axial_DIN0309_L9.0mm_D3.2mm_P12.70mm_Horizontal" (id 2) (at 260.858 102.87 90)
+    (property "Footprint" "Resistor_THT:R_Axial_DIN0309_L9.0mm_D3.2mm_P15.24mm_Horizontal" (id 2) (at 260.858 102.87 90)
       (effects (font (size 1.27 1.27)) hide)
     )
@@
       (effects (font (size 1.27 1.27)) (justify right))
     )
-    (property "Footprint" "Resistor_THT:R_Axial_DIN0309_L9.0mm_D3.2mm_P12.70mm_Horizontal" (id 2) (at 260.858 83.82 90)
+    (property "Footprint" "Resistor_THT:R_Axial_DIN0309_L9.0mm_D3.2mm_P15.24mm_Horizontal" (id 2) (at 260.858 83.82 90)
       (effects (font (size 1.27 1.27)) hide)
     )
@@
     )
     (path "/4b6ececa-1c47-49b9-9721-c1891674c6db"
-      (reference "R18") (unit 1) (value "R10K") (footprint "Resistor_THT:R_Axial_DIN0309_L9.0mm_D3.2mm_P12.70mm_Horizontal")
+      (reference "R18") (unit 1) (value "R10K") (footprint "Resistor_THT:R_Axial_DIN0309_L9.0mm_D3.2mm_P15.24mm_Horizontal")
     )
     (path "/417c4c24-c305-41be-8348-76e7579feb15"
@@
     )
     (path "/426a62f8-cf65-48b3-9dac-dadeff6e3f1b"
-      (reference "R20") (unit 1) (value "R10K") (footprint "Resistor_THT:R_Axial_DIN0309_L9.0mm_D3.2mm_P12.70mm_Horizontal")
+      (reference "R20") (unit 1) (value "R10K") (footprint "Resistor_THT:R_Axial_DIN0309_L9.0mm_D3.2mm_P15.24mm_Horizontal")
     )
     (path "/14ec2fba-b378-4d0b-b95a-ec2ddf937961"

Commit message: Network finished
Parts:
- R16: footprint Resistor_THT:R_Axial_DIN0309_L9.0mm_D3.2mm_P12.70mm_Horizontal -> Resistor_THT:R_Axial_DIN0309_L9.0mm_D3.2mm_P15.24mm_Horizontal
Changed lines of the file:
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@@
       (effects (font (size 1.27 1.27)) (justify right))
     )
-    (property "Footprint" "Resistor_THT:R_Axial_DIN0309_L9.0mm_D3.2mm_P12.70mm_Horizontal" (id 2) (at 260.858 62.23 90)
+    (property "Footprint" "Resistor_THT:R_Axial_DIN0309_L9.0mm_D3.2mm_P15.24mm_Horizontal" (id 2) (at 260.858 62.23 90)
       (effects (font (size 1.27 1.27)) hide)
     )
@@
     )
     (path "/7896e020-a247-4952-982c-204414362fdb"
-      (reference "R16") (unit 1) (value "R10K") (footprint "Resistor_THT:R_Axial_DIN0309_L9.0mm_D3.2mm_P12.70mm_Horizontal")
+      (reference "R16") (unit 1) (value "R10K") (footprint "Resistor_THT:R_Axial_DIN0309_L9.0mm_D3.2mm_P15.24mm_Horizontal")
     )
     (path "/c4ba95a0-8610-4ffa-972a-bb866f65968c"
