File: retro-game-console.kicad_pcb (KiCad board)
At the start: 2 copper layers, 96.5 x 137.2 mm, 42 parts, among them J1 Battery_Clip, U1 ESP32-DevKitC, U2 Battery_shield_v3, U3 Micro_SD_card_adapter, U4 MAX98357A_Breakout, U5 LCD_ILI9341, U6 74HC165

Commit message: Before net
Parts:
- R13, R14, R15, R18, R20: moved to F.Cu
- moved U2 405.0 mm to (-351.9, 158.8)
- moved U5 399.6 mm to (-296.3, 49.6)
- moved R2 382.7 mm to (-275.6, 88.9), turned to 180 degrees
- moved R9 360.0 mm to (-275.6, 78.7), turned to 180 degrees
- moved R3 320.9 mm to (-275.6, 68.6), turned to 180 degrees
- moved R20 309.3 mm to (-191.8, 226.1)
- moved SW_A1 307.4 mm to (-204.4, 203.2)
- moved R18 302.7 mm to (-191.8, 190.5)
- moved SW_B1 300.9 mm to (-204.4, 236.3)
- moved R11 299.9 mm to (-215.9, 85.1), turned to -90 degrees
- moved LS1 299.7 mm to (-223.5, 30.5), turned to 90 degrees
- moved R12 285.1 mm to (-222.2, -15.2), turned to 0 degrees
- moved R8 278.5 mm to (-224.8, -25.4), turned to 0 degrees
- moved R10 275.5 mm to (-222.2, -5.08), turned to 0 degrees
- moved C2 273.4 mm to (-220.9, -35.6), turned to 0 degrees
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Connections:
- D1 pad 1: Net-(D1-Pad1) -> GND
- D1 pad 2: LED_PIN -> Net-(D1-Pad2)
- R1 pad 1: Net-(D1-Pad1) -> LED_PIN
- R1 pad 2: GND -> Net-(D1-Pad2)
Routing:
- net GND: track 340.2 -> 0.00 mm, vias 6 -> 0
- net +3.3V: track 294.4 -> 0.00 mm
- net Net-(LS1-Pad2): track 66.4 -> 0.00 mm
- net Net-(LS1-Pad1): track 62.1 -> 0.00 mm
- net BAT_LEVEL: track 50.6 -> 0.00 mm
- net BTN_A: track 29.8 -> 0.00 mm
- net BTN_START: track 26.8 -> 0.00 mm, vias 1 -> 0
- net BTN_OPTION: track 23.2 -> 0.00 mm
- net BTN_RIGHT: track 19.7 -> 0.00 mm
- net BTN_SELECT: track 17.2 -> 0.00 mm, vias 1 -> 0
- net BTN_LEFT: track 16.8 -> 0.00 mm
- net BTN_UP: track 16.7 -> 0.00 mm
- net BTN_DOWN: track 16.7 -> 0.00 mm
- net Net-(J1-Pad1): track 16.3 -> 0.00 mm
- net Net-(R6-Pad1): track 15.9 -> 0.00 mm
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
Commit message: WIP
Parts:
- C1, C2, C3, J1, R6, R7, R8: moved to F.Cu
- LS1, R1, R13, R14, R15, R16, R17, R19, R2, R4, R5, R9, U4: moved to B.Cu
- R18, R20: footprint Resistor_THT:R_Axial_DIN0309_L9.0mm_D3.2mm_P12.70mm_Horizontal -> Resistor_THT:R_Axial_DIN0309_L9.0mm_D3.2mm_P15.24mm_Horizontal; moved to B.Cu
- moved U5 399.5 mm to (101.6, 14.1)
- moved R3 373.3 mm to (96.5, 97.8), turned to -90 degrees
- moved U2 363.4 mm to (11.4, 148.7), turned to 0 degrees
- moved R2 359.5 mm to (81.3, 45.7), turned to 0 degrees
- moved R9 359.2 mm to (81.3, 38.1), turned to 0 degrees
- moved R12 321.5 mm to (73.7, 110.5), turned to 90 degrees
- moved R10 320.5 mm to (81.3, 97.8), turned to -90 degrees
- moved SW_A1 317.0 mm to (103.9, 129.5), turned to 180 degrees
- moved SW_B1 309.5 mm to (86.2, 129.5), turned to 180 degrees
- moved R11 305.1 mm to (88.9, 97.8)
- moved C2 299.8 mm to (45.6, 101.6), turned to 180 degrees
- moved R18 294.7 mm to (97.6, 134.6), turned to 90 degrees
- moved R20 286.7 mm to (79.9, 134.6), turned to 90 degrees
- moved R8 273.8 mm to (17.8, 101.6)
- moved R7 271.6 mm to (48.3, 94.0), turned to 180 degrees
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
Commit message: Network finished
Parts:
- R16: footprint Resistor_THT:R_Axial_DIN0309_L9.0mm_D3.2mm_P12.70mm_Horizontal -> Resistor_THT:R_Axial_DIN0309_L9.0mm_D3.2mm_P15.24mm_Horizontal
- moved R18 14.6 mm to (97.9, 120.0), turned to -90 degrees
- moved R20 14.6 mm to (80.1, 120.0), turned to -90 degrees
- moved SW_A1 13.2 mm to (91.5, 125.1), turned to 0 degrees
- moved SW_B1 13.1 mm to (73.8, 125.1), turned to 0 degrees
- moved R19 12.4 mm to (67.4, 133.7), turned to -90 degrees
- moved R17 12.4 mm to (56.0, 133.7), turned to -90 degrees
- moved R9 5.08 mm to (81.3, 33.0)
- moved U6 3.60 mm to (63.7, 118.8)
- moved D1 2.92 mm to (19.3, 17.3), turned to 180 degrees
- moved R16 1.36 mm to (43.4, 120.0)
- moved C2 1.34 mm to (44.4, 102.2)
- moved R10 1.34 mm to (80.1, 98.4)
- moved R11 1.34 mm to (87.7, 98.4)
- moved R12 1.34 mm to (72.5, 111.1)
- moved R13 1.34 mm to (33.2, 122.6)
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Routing:
- net GND: track 0.00 -> 583.1 mm, vias 0 -> 6
- net +3.3V: track 0.00 -> 443.1 mm, vias 0 -> 8
- net BTN_LEFT: track 0.00 -> 96.7 mm, vias 0 -> 2
- net LCD_BCKL_OUT: track 0.00 -> 86.1 mm
- net LCD_SCK: track 0.00 -> 85.0 mm, vias 0 -> 2
- net BTN_DOWN: track 0.00 -> 83.9 mm, vias 0 -> 2
- net LCD_MOSI: track 0.00 -> 77.6 mm
- net Net-(D1-Pad2): track 0.00 -> 72.2 mm
- net BTN_B: track 0.00 -> 69.7 mm, vias 0 -> 2
- net BTN_OPTION: track 0.00 -> 56.3 mm, vias 0 -> 1
- net BTN_A: track 0.00 -> 56.1 mm, vias 0 -> 2
- net LCD_CS: track 0.00 -> 48.1 mm
- net AUD_LRC: track 0.00 -> 46.4 mm
- net Net-(LS1-Pad2): track 0.00 -> 45.0 mm
- net BTN_RIGHT: track 0.00 -> 44.9 mm
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
Commit message: Fix
Routing:
- net Net-(LS1-Pad2): track 45.0 -> 47.6 mm
- net LCD_MOSI: track 77.6 -> 76.6 mm
- net Net-(LS1-Pad1): track 29.9 -> 30.8 mm
- net LCD_SCK: track 85.0 -> 84.4 mm
Changed lines of the file:
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@@
   (segment (start 53.75656 63.5) (end 53.75656 66.45656) (width 1) (layer "B.Cu") (net 4))
   (segment (start 17.78 88.9) (end 17.78 93.98) (width 1) (layer "B.Cu") (net 5))
-  (segment (start 20.32 40.64) (end 21.081999 41.401999) (width 1) (layer "B.Cu") (net 6))
-  (segment (start 21.081999 41.401999) (end 21.081999 68.692564) (width 1) (layer "B.Cu") (net 6))
-  (segment (start 21.081999 68.692564) (end 19.986545 69.788018) (width 1) (layer "B.Cu") (net 6))
-  (segment (start 16.375076 34.424924) (end 16.375076 68.716549) (width 1) (layer "B.Cu") (net 7))
-  (segment (start 16.375076 68.716549) (end 19.986545 72.328018) (width 1) (layer "B.Cu") (net 7))
-  (segment (start 20.32 30.48) (end 16.375076 34.424924) (width 1) (layer "B.Cu") (net 7))
+  (segment (start 22.1097 67.664863) (end 19.986545 69.788018) (width 1) (layer "B.Cu") (net 6))
+  (segment (start 22.1097 42.4297) (end 22.1097 67.664863) (width 1) (layer "B.Cu") (net 6))
+  (segment (start 20.32 40.64) (end 22.1097 42.4297) (width 1) (layer "B.Cu") (net 6))
+  (segment (start 17.881759 72.328018) (end 19.986545 72.328018) (width 1) (layer "B.Cu") (net 7))
+  (segment (start 14.695227 36.104773) (end 14.695227 69.141486) (width 1) (layer "B.Cu") (net 7))
+  (segment (start 14.695227 69.141486) (end 17.881759 72.328018) (width 1) (layer "B.Cu") (net 7))
+  (segment (start 20.32 30.48) (end 14.695227 36.104773) (width 1) (layer "B.Cu") (net 7))
   (segment (start 95.050524 44.649476) (end 93.98 45.72) (width 1) (layer "B.Cu") (net 8))
   (segment (start 99.781579 44.649476) (end 95.050524 44.649476) (width 1) (layer "B.Cu") (net 8))
@@
   (segment (start 95.329557 98.410261) (end 93.330261 98.410261) (width 1) (layer "B.Cu") (net 9))
   (segment (start 71.53656 89.31656) (end 71.53656 88.9) (width 1) (layer "B.Cu") (net 9))
-  (segment (start 95.329557 104.760261) (end 95.329557 111.110261) (width 1) (layer "B.Cu") (net 10))
-  (segment (start 106.68 38.1) (end 106.68 86.36) (width 1) (layer "B.Cu") (net 10))
   (segment (start 102.949557 97.140261) (end 95.329557 104.760261) (width 1) (layer "B.Cu") (net 10))
-  (segment (start 103.069476 34.489476) (end 106.68 38.1) (width 1) (layer "B.Cu") (net 10))
   (segment (start 106.68 86.36) (end 102.949557 90.090443) (width 1) (layer "B.Cu") (net 10))
   (segment (start 102.949557 90.090443) (end 102.949557 97.140261) (width 1) (layer "B.Cu") (net 10))
-  (segment (start 99.781579 34.489476) (end 103.069476 34.489476) (width 1) (layer "B.Cu") (net 10))
+  (segment (start 106.68 38.279536) (end 106.68 86.36) (width 1) (layer "B.Cu") (net 10))
+  (segment (start 102.88994 34.489476) (end 106.68 38.279536) (width 1) (layer "B.Cu") (net 10))
+  (segment (start 95.329557 104.760261) (end 95.329557 111.110261) (width 1) (layer "B.Cu") (net 10))
+  (segment (start 99.781579 34.489476) (end 102.88994 34.489476) (width 1) (layer "B.Cu") (net 10))
   (segment (start 92.545 68.29) (end 91.73 68.29) (width 1) (layer "F.Cu") (net 11))
   (segment (start 94.9875 71.12) (end 97.665 71.12) (width 1) (layer "F.Cu") (net 11))
@@
   (segment (start 34.033263 63.417618) (end 31.820997 63.417618) (width 1) (layer "B.Cu") (net 35))
   (segment (start 66.45656 86.77656) (end 55.88 76.2) (width 1) (layer "B.Cu") (net 35))
-  (segment (start 104.14 55.88) (end 104.14 38.1) (width 1) (layer "F.Cu") (net 36))
-  (segment (start 101.6 58.42) (end 104.14 55.88) (width 1) (layer "F.Cu") (net 36))
-  (via (at 104.14 38.1) (size 1) (drill 0.4) (layers "F.Cu" "B.Cu") (net 36))
+  (segment (start 104.14 39.249493) (end 104.14 55.88) (width 1) (layer "F.Cu") (net 36))
+  (segment (start 104.14 55.88) (end 101.6 58.42) (width 1) (layer "F.Cu") (net 36))
+  (via (at 104.14 39.249493) (size 1) (drill 0.4) (layers "F.Cu" "B.Cu") (net 36))
   (via (at 101.6 58.42) (size 1) (drill 0.4) (layers "F.Cu" "B.Cu") (net 36))
+  (segment (start 104.14 39.249493) (end 101.919983 37.029476) (width 1) (layer "B.Cu") (net 36))
   (segment (start 68.99656 88.48344) (end 75.282086 82.197914) (width 1) (layer "B.Cu") (net 36))
   (segment (start 101.6 81.28) (end 101.6 58.42) (width 1) (layer "B.Cu") (net 36))
   (segment (start 75.282086 82.197914) (end 100.682086 82.197914) (width 1) (layer "B.Cu") (net 36))
   (segment (start 68.99656 88.9) (end 68.99656 88.48344) (width 1) (layer "B.Cu") (net 36))
-  (segment (start 99.781579 37.029476) (end 103.069476 37.029476) (width 1) (layer "B.Cu") (net 36))
   (segment (start 100.682086 82.197914) (end 101.6 81.28) (width 1) (layer "B.Cu") (net 36))
-  (segment (start 104.14 38.1) (end 103.069476 37.029476) (width 1) (layer "B.Cu") (net 36))
-  (segment (start 104.14 40.64) (end 104.14 83.82) (width 1) (layer "B.Cu") (net 38))
+  (segment (start 101.919983 37.029476) (end 99.781579 37.029476) (width 1) (layer "B.Cu") (net 36))
+  (segment (start 104.14 42.440022) (end 104.14 83.82) (width 1) (layer "B.Cu") (net 38))
+  (segment (start 104.14 83.82) (end 102.758003 85.201997) (width 1) (layer "B.Cu") (net 38))
+  (segment (start 101.269454 39.569476) (end 104.14 42.440022) (width 1) (layer "B.Cu") (net 38))
   (segment (start 102.758003 85.201997) (end 80.314563 85.201997) (width 1) (layer "B.Cu") (net 38))
+  (segment (start 99.781579 39.569476) (end 101.269454 39.569476) (width 1) (layer "B.Cu") (net 38))
   (segment (start 80.314563 85.201997) (end 76.61656 88.9) (width 1) (layer "B.Cu") (net 38))
-  (segment (start 104.14 83.82) (end 102.758003 85.201997) (width 1) (layer "B.Cu") (net 38))
-  (segment (start 103.069476 39.569476) (end 104.14 40.64) (width 1) (layer "B.Cu") (net 38))
-  (segment (start 99.781579 39.569476) (end 103.069476 39.569476) (width 1) (layer "B.Cu") (net 38))
   (segment (start 99.781579 47.189476) (end 97.590524 47.189476) (width 1) (layer "B.Cu") (net 46))
   (segment (start 88.9 45.72) (end 88.9 41.875763) (width 1) (layer "B.Cu") (net 46))
