File: retro-game-console.kicad_pcb (KiCad board)
At the start: 2 copper layers, 96.5 x 137.2 mm, 42 parts, among them J1 Battery_Clip, U1 ESP32-DevKitC, U2 Battery_shield_v3, U3 Micro_SD_card_adapter, U4 MAX98357A_Breakout, U5 LCD_ILI9341, U6 74HC165

Commit message: Final v1
Routing:
- net GND: track 582.7 -> 573.1 mm, vias 6 -> 8
- net BTN_START: track 39.9 -> 44.8 mm, vias 1 -> 3
- net BTN_DOWN: track 83.9 -> 86.9 mm
- net BTN_RIGHT: track 44.9 -> 47.5 mm
- net Net-(R10-Pad2): track 21.8 -> 19.6 mm
- net BTN_LEFT: track 96.7 -> 95.3 mm, vias 2 -> 3
- net +3.3V: track 443.1 -> 441.9 mm, vias 8 -> 6
- net Net-(R11-Pad2): track 32.4 -> 31.3 mm
- net BTN_B: track 69.7 -> 70.8 mm
- net BTN_SELECT: track 44.3 -> 45.3 mm, vias 1 -> 3

Commit message: Final v1.1
Parts:
- moved R9 7.67 mm to (81.2, 40.7)
Routing:
- net GND: track 573.1 -> 541.8 mm, vias 8 -> 7
- net LCD_CS: track 48.1 -> 34.2 mm, vias 0 -> 2
- net LCD_DC: track 32.4 -> 24.7 mm
- net LCD_DC_OUT: track 14.0 -> 6.47 mm
- net SD_MISO: track 16.5 -> 11.4 mm, vias 2 -> 1
- net LCD_SCK: track 84.4 -> 89.4 mm
- net SD_CS: track 14.2 -> 16.9 mm, vias 0 -> 1
- net LCD_BCKL_OUT: track 86.0 -> 87.6 mm
- net SD_MOSI: track 26.0 -> 27.1 mm, vias 0 -> 1
- net Net-(LS1-Pad2): track 47.6 -> 46.5 mm
- net LCD_MOSI: track 76.6 -> 77.6 mm
- net Net-(LS1-Pad1): track 30.8 -> 31.5 mm
- net AUD_BCLK: track 42.8 -> 42.7 mm, vias 0 -> 1
- net SD_SCK: track 11.5 -> 11.7 mm, vias 0 -> 1
- net AUD_DIN: vias 0 -> 1
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
Commit message: snapshot
Routing:
- net BTN_SELECT: vias 3 -> 2
Changed lines of the file:
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@@
   (segment (start 67.784514 125.255486) (end 67.784514 114.920261) (width 1) (layer "F.Cu") (net 26))
   (segment (start 52.012772 137.780261) (end 53.304908 136.488125) (width 1) (layer "F.Cu") (net 26))
-  (via (at 60.96 132.08) (size 1) (drill 0.4) (layers "F.Cu" "B.Cu") (net 26))
   (via (at 67.784514 114.920261) (size 1) (drill 0.4) (layers "F.Cu" "B.Cu") (net 26))
   (via (at 60.96 132.08) (size 1) (drill 0.4) (layers "F.Cu" "B.Cu") (net 26))
